File: hardware/line.kicad_pcb (KiCad board)
At the start: 2 copper layers, 25 x 15 mm, 12 parts, among them P1 CON-SENSOR, Q1 2N7002P, U1 M24C64, U2 CNY70, U3 DRILL, U4 DRILL

Commit message: Add 3d information (tbc)
Parts:
- C1: footprint 0603 -> C0603
- R1: footprint 0603 -> R0603
- VAL: footprint WEEE_7mm -> kicad-libraries:WEEE_7mm
- VAL: footprint CE_5mm -> kicad-libraries:CE_5mm
Connections:
- P1 pad 10: (no net) -> Net-(P1-Pad10)
- P1 pad 9: (no net) -> Net-(P1-Pad9)
- RP1 pad 2: (no net) -> Net-(RP1-Pad2)
- RP1 pad 3: (no net) -> Net-(RP1-Pad3)
- U1 pad 7: (no net) -> Net-(U1-Pad7)
